File: WetProgrammer.kicad_pcb (KiCad board)
At the start: 2 copper layers, 48 x 25 mm, 33 parts, among them J1 USB_B_Micro, SW1 SW_SPDT, U1 ATmega32U4-AU, U2 TLV1117-33, Y1 16MHz

Commit message: Changes as requested by Ben
Parts:
- removed JP4: Jumper_2_Open, Connector_PinHeader_2.54mm:PinHeader_1x02_P2.54mm_Vertical
- added FID1: Fiducial, Fiducial:Fiducial_1mm_Mask2mm, F.Cu at (2.00, -2.00)
- added FID2: Fiducial, Fiducial:Fiducial_1mm_Mask2mm, F.Cu at (46.0, -23.0)
- added H1: MountingHole, MountingHole:MountingHole_3.2mm_M3, F.Cu at (45.5, -2.50)
- added H2: MountingHole, MountingHole:MountingHole_3.2mm_M3, F.Cu at (2.50, -22.5)
- added J3: Conn_01x03_Male, Connector_PinHeader_2.54mm:PinHeader_1x03_P2.54mm_Vertical, F.Cu at (39.4, -8.64)
- added R10: 330, Resistor_SMD:R_0805_2012Metric, F.Cu at (35.8, -2.79)
- added R11: 330, Resistor_SMD:R_0805_2012Metric, F.Cu at (35.8, -4.76)
- added SW2: SW_SPDT, tmc:388Switch, F.Cu at (39.8, -23.0)
- moved R7 6.41 mm to (31.6, -8.32), turned to 270 degrees
- moved R9 4.83 mm to (33.7, -8.32), turned to 270 degrees
- moved R8 4.77 mm to (35.8, -8.29), turned to 270 degrees
- moved D1 4.40 mm to (36.3, -18.0), turned to 180 degrees
- moved R6 4.35 mm to (39.3, -15.2)
- moved C8 2.52 mm to (23.5, -21.0)
- moved C7 2.36 mm to (21.3, -21.0)
- moved SW1 1.50 mm to (10.0, -23.0)
- moved C3 1.40 mm to (19.2, -21.0), turned to 270 degrees
- moved U2 1.14 mm to (30.0, -20.5)
- moved JP1 0.50 mm to (16.7, -21.0)
- moved C1 0.10 mm to (33.0, -3.90)
- renumbered DUT to J2, 32u4 to JPROG1
Routing:
- net +3V3: track 26.7 -> 0.00 mm
- net VBUS: track 36.1 -> 10.9 mm, vias 2 -> 0
- net Net-(R10-Pad2): track 0.00 -> 15.3 mm
- net VCC: track 81.2 -> 66.3 mm
- net Net-(R11-Pad2): track 0.00 -> 14.3 mm
- net GND: track 27.1 -> 15.4 mm, vias 26 -> 21
- net /TXO: track 0.00 -> 8.46 mm
- net /MISO: track 35.9 -> 30.1 mm
- net Net-(J2-Pad1): track 8.58 -> 13.9 mm
- net Net-(C3-Pad2): track 4.63 -> 0.00 mm
- net /SCK: track 35.1 -> 31.8 mm
- net /RXI: track 0.00 -> 3.19 mm
- net Net-(J2-Pad3): track 8.14 -> 10.8 mm
- net Net-(R6-Pad2): track 13.5 -> 15.9 mm
- net /VProg: track 6.77 -> 8.96 mm
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Other:
- board text added: "3v3"
- board text added: "5"
- board text added: "Rev 1.0, Sep 2021 github.com/timChase98/WetAvrProgrammer"
- board text added: "T-> R<- Gnd"
- board text added: "W.E.T. AVR Programmer Tim Chase"
- board text removed: "+3V3"
- board text removed: "+5V"
- board text removed: "Xplained Programmer Schematic and Layout by Tim Chase For the University of Massachusetts Dartmouth Rev 1.0, Sep 2021 https://github.com/timChase98/WetAvrProgrammer"

Commit message: Connected swtich sheilding to gnd
Parts:
- moved C8 0.56 mm to (24.0, -21.3)
- moved C7 0.35 mm to (21.6, -21.3)
- moved C3 0.25 mm to (19.2, -21.3)
Connections:
- SW1 pad 6: (no net) -> GND
- SW2 pad 6: (no net) -> GND
Routing:
- net +3V3: track 0.00 -> 30.9 mm
- net VBUS: track 10.9 -> 40.6 mm
- net GND: track 15.4 -> 29.2 mm, vias 21 -> 27
- net VCC: track 66.3 -> 77.7 mm
- net Net-(C3-Pad2): track 0.00 -> 4.70 mm
Other:
- board text added: "ON"
